File: maXTouch Xplained Shield.brd (EAGLE design)
At the start: 51.8 x 69.3 mm, 10 parts, among them IC1 MIC29502BT

Commit message: THandSMD
Parts:
- added C3: 100uF, SparkFun-Capacitors:CPOL-RADIAL-2.5MM-6.5MM
- added C4: 0.1uF, SparkFun-Capacitors:CAP-PTH-SMALL-KIT
- added R3: 160R, SparkFun-Resistors:AXIAL-0.3-KIT
- added R4: 100R, SparkFun-Resistors:AXIAL-0.3-KIT
- C2: device SparkFun-Capacitors:0805 -> SparkFun-Capacitors:1206
- R1, R2: device SparkFun-Resistors:0603 -> SparkFun-Resistors:1206
- moved R1 9.75 mm to (25.4, 34.8), turned to 270 degrees
- moved IC1 8.39 mm to (26.0, 22.5)
- moved C2 6.40 mm to (19.1, 37.8), turned to 270 degrees
- moved C1 6.23 mm to (27.2, 51.1)
- moved R2 5.25 mm to (21.6, 34.8)
- moved J3 5.08 mm to (28.5, 56.3)
- moved J5 2.83 mm to (33.6, 58.8)
Connections:
- net 3V3: now also C4.1, R3.P$2
- net 5V: now also C3.1
- net GND: now also C3.2, C4.2, R4.P$1
- net N$2: now also R3.P$1, R4.P$2
Routing:
- net 5V: track 28.1 -> 43.8 mm
- net 3V3: track 19.3 -> 34.8 mm
- net PWM: track 44.4 -> 59.1 mm
- net CS: track 22.7 -> 30.6 mm
- net SDA: track 36.5 -> 44.0 mm
- net RST: track 63.3 -> 69.7 mm
- net N$2: track 7.42 -> 12.9 mm
- net MISO: track 16.7 -> 21.7 mm
- net MOSI: track 21.7 -> 26.8 mm
- net SCK: track 54.3 -> 50.5 mm
- net SCL: track 48.9 -> 47.9 mm
